File: PPS-Power-Supply.kicad_pcb (KiCad board)
At the start: 4 copper layers, 94.2 x 52.3 mm, 98 parts, among them J1 USB_C_Receptacle_PowerOnly_6P, J10 VBUS, J2 GMT130-V1.0, J3 SPI2, J4 GPIOs, J5 GPIOs, J6 DEBUG, J8 PJ-002AH, J9 GND, U1 STM32G071KBTxN, U2 TCPP01-M12, U3 RT8250, U4 INA219AxD, U5 TLV9001IDCK, U6 STL11N3LLH6, U7 Joystick, Y1 32.768 kHz

Commit message: updated
Parts:
- added G***: LOGO, LOGO, F.Cu at (221.3, 92.5)
- added G***: LOGO, LOGO, B.Cu at (176.3, 75.8)
- D3: footprint Diode_SMD:D_SMA -> Diode_SMD:D_SMB
Routing:
- net VBUS: vias 15 -> 16
