File: PPS-Power-Supply.kicad_sch (KiCad schematic)
At the start: 97 parts, among them J1 USB_C_Receptacle_PowerOnly_6P, J10 VBUS, J2 GMT130-V1.0, J3 SPI2, J4 GPIOs, J5 GPIOs, J6 DEBUG, J8 PJ-002AH, J9 GND, U1 STM32G071KBTxN, U2 TCPP01-M12, U3 RT8250, U4 INA219AxD, U5 TLV9001IDCK, U6 STL11N3LLH6, U7 Joystick, Y1 32.768 kHz

Commit message: updated
Parts:
- D3: footprint Diode_SMD:D_SMA -> Diode_SMD:D_SMB
Connections:
- no-connect marks 2 -> 1
Other:
- note removed: "KÖP: BAT54J (och BAT54K kanske) TCPP01 N-MOSFET - STL11N3LLH6 STM32 TLV9001 op amp FC-135R 32.7680KA-AC0 C1F 7 (FUSE) SMBJ24A (TVS) PJ-002AH (Barrel jack) 10 ohm (0603) 30-50 st 82k ohm (0603) 20-30 st 26k1 ohm (0603) 20-30 st 6k8 ohm (0603) 20-30 st 620 ohm (0603) 20-30 st Dubbelkolla om du har spole 1206 10uF cap 0603 3n9 cap 0805 4u7 cap SRN5040TA-100M 10mOHM resistor shunt 3W"
Changed lines of the file:
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@@
 		)
 	)
-	(text "KÖP:\nBAT54J (och BAT54K kanske)\nTCPP01\nN-MOSFET - STL11N3LLH6\nSTM32\nTLV9001 op amp\nFC-135R 32.7680KA-AC0 \nC1F 7  (FUSE)\nSMBJ24A (TVS)\nPJ-002AH (Barrel jack)\n10 ohm (0603) 30-50 st\n82k ohm (0603) 20-30 st\n26k1 ohm (0603) 20-30 st\n6k8 ohm (0603) 20-30 st\n620 ohm (0603) 20-30 st\nDubbelkolla om du har spole\n1206 10uF cap\n0603 3n9 cap\n0805 4u7 cap\nSRN5040TA-100M \n10mOHM resistor shunt 3W"
-		(exclude_from_sim no)
-		(at -38.1 114.554 0)
-		(effects
-			(font
-				(size 1.27 1.27)
-				(thickness 0.254)
-				(bold yes)
-			)
-			(justify left)
-		)
-	)
 	(text ""
 		(exclude_from_sim no)
@@
 		)
 	)
-	(text "CHECK FOOTPRINT"
-		(exclude_from_sim no)
-		(at 42.672 56.388 0)
-		(effects
-			(font
-				(size 1.27 1.27)
-			)
-		)
-	)
 	(text "Figure 13 in datasheet"
 		(exclude_from_sim no)
@@
 	)
 	(no_connect
-		(at 162.56 127)
-	)
-	(no_connect
 		(at 259.08 124.46)
 	)
@@
 			)
 		)
-		(property "Footprint" "Diode_SMD:D_SMA"
+		(property "Footprint" "Diode_SMD:D_SMB"
 			(at 38.1 55.88 0)
 			(hide yes)
